File: GNSS.kicad_sch (KiCad schematic)
At the start: 5 parts, among them U6 Teseo-LIV3FL

Commit message: update output files for v1.0
Other:
- company: (none) -> Domonic Richardson
- title: (none) -> LoRa Tracker HAT+ - GNSS Module
Changed lines of the file:
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@@
 	(generator_version "9.0")
 	(paper "A4")
+	(title_block
+		(title "LoRa Tracker HAT+ - GNSS Module")
+		(date "2025-07-05")
+		(rev "v1.0")
+		(company "Domonic Richardson")
+	)
 	(junction
 		(at 140.97 119.38)
