File: LoRa.kicad_sch (KiCad schematic)
At the start: 37 parts, among them U3 SX1272, U4 NC7SZ04P5X, U5 AS222-92LF, X2 32MHz

Commit message: update output files for v1.0
Other:
- company: (none) -> Domonic Richardson
- title: (none) -> LoRa Tracker HAT+ - LoRa Transceiver and Matching Network
Changed lines of the file:
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@@
 	(generator_version "9.0")
 	(paper "A4")
+	(title_block
+		(title "LoRa Tracker HAT+ - LoRa Transceiver and Matching Network")
+		(date "2025-07-05")
+		(rev "v1.0")
+		(company "Domonic Richardson")
+	)
 	(text "Bulk Decoupling"
 		(exclude_from_sim no)
