File: RPi.kicad_sch (KiCad schematic)
At the start: 11 parts, among them U2 CAT24C32WI-GT3

Commit message: update output files for v1.0
Other:
- company: (none) -> Domonic Richardson
- title: (none) -> LoRa Tracker HAT+ - RPi Connections
Changed lines of the file:
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@@
 	(generator_version "9.0")
 	(paper "A4")
+	(title_block
+		(title "LoRa Tracker HAT+ - RPi Connections")
+		(date "2025-07-05")
+		(rev "v1.0")
+		(company "Domonic Richardson")
+	)
 	(rectangle
 		(start 71.12 53.34)
