File: loratracker_hat.kicad_sch (KiCad schematic)
At the start: 41 parts, among them SW1 RESET, SW2 BTN2, SW3 BTN1, U1 STM32H7B0RBTx, X1 25MHz

Commit message: update output files for v1.0
Other:
- title: LoRa Tracking HAT -> LoRa Tracker HAT+ - uC and User Interface
Changed lines of the file:
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@@
 	(paper "A4")
 	(title_block
-		(title "LoRa Tracking HAT")
+		(title "LoRa Tracker HAT+ - uC and User Interface")
 		(date "2025-07-05")
-		(rev "v1")
+		(rev "v1.0")
 		(company "Domonic Richardson")
 	)
@@
 		)
 		(instances
-			(project "anchor_node"
+			(project "loratracker_hat"
 				(path "/51073acf-2ecf-4a2e-adb3-f8c43b45512e"
 					(page "2")
@@
 		)
 		(instances
-			(project "anchor_node"
+			(project "loratracker_hat"
 				(path "/51073acf-2ecf-4a2e-adb3-f8c43b45512e"
 					(page "3")
@@
 		)
 		(instances
-			(project "anchor_node"
+			(project "loratracker_hat"
 				(path "/51073acf-2ecf-4a2e-adb3-f8c43b45512e"
 					(page "4")
